Commit message: ranger gazebo only, but wheel odom must be modiefied

File: gazebo_ranger/urdf/ranger_mini.xacro (robot description, xacro)
@@ -537,5 +537,5 @@
   <gazebo>
     <plugin filename="libgazebo_ros2_control.so" name="gazebo_ros2_control">
-      <parameters>$(find gazebo_ranger)/config/controller.yaml</parameters>
+      <parameters>$(find gazebo_ranger)/config/config.yaml</parameters>
     </plugin>
   </gazebo>

File: gazebo_ranger/urdf/sensors/gps.xacro (robot description, xacro)
@@ -2,7 +2,7 @@
 <robot xmlns:xacro="http://www.ros.org/wiki/xacro" name="gps">
     <xacro:property name="M_PI" value="3.1415926535897931" />
-    <xacro:macro name="gps" params="path:='$(find gazebo_ranger)/config/sensor_params.yaml'">
+    <xacro:macro name="gps" params="path:='$(find gazebo_ranger)/config/config.yaml'">
     <!-- Extracting values from the params -->
-    <xacro:property name="yaml_path" value="$(find gazebo_ranger)/config/sensor_params.yaml" />
+    <xacro:property name="yaml_path" value="$(find gazebo_ranger)/config/config.yaml" />
     <xacro:property name="dict_yaml" value="${xacro.load_yaml(yaml_path)}" />
     <xacro:property name="gps" value="${dict_yaml['gps']}" />

File: gazebo_ranger/urdf/sensors/imu.xacro (robot description, xacro)
@@ -2,7 +2,7 @@
 <robot xmlns:xacro="http://www.ros.org/wiki/xacro" name="imu">
     <xacro:property name="M_PI" value="3.1415926535897931" />
-    <xacro:macro name="imu" params="path:='$(find gazebo_ranger)/config/sensor_params.yaml'">
+    <xacro:macro name="imu" params="path:='$(find gazebo_ranger)/config/config.yaml'">
     <!-- Extracting values from the params -->
-    <xacro:property name="yaml_path" value="$(find gazebo_ranger)/config/sensor_params.yaml" />
+    <xacro:property name="yaml_path" value="$(find gazebo_ranger)/config/config.yaml" />
     <xacro:property name="dict_yaml" value="${xacro.load_yaml(yaml_path)}" />
     <xacro:property name="imu" value="${dict_yaml['imu']}" />

File: gazebo_ranger/urdf/sensors/kinect_camera.xacro (robot description, xacro)
@@ -4,5 +4,5 @@
   <xacro:macro name="kinect_camera" params="camera_key:='camera'">
     <!-- Extracting values from the params -->
-    <xacro:property name="yaml_path" value="$(find gazebo_ranger)/config/sensor_params.yaml" />
+    <xacro:property name="yaml_path" value="$(find gazebo_ranger)/config/config.yaml" />
     <xacro:property name="dict_yaml" value="${xacro.load_yaml(yaml_path)}" />
     <xacro:property name="camera" value="${dict_yaml[camera_key]}" />

File: gazebo_ranger/urdf/sensors/vlp-32.urdf.xacro (robot description, xacro)
@@ -3,5 +3,5 @@
   <xacro:property name="M_PI" value="3.1415926535897931" />
   <xacro:macro name="VLP-32" params="*origin">
-  <xacro:property name="yaml_path" value="$(find gazebo_ranger)/config/sensor_params.yaml" />
+  <xacro:property name="yaml_path" value="$(find gazebo_ranger)/config/config.yaml" />
   <xacro:property name="dict_yaml" value="${xacro.load_yaml(yaml_path)}" />
   <!-- lidar parameters -->
